File: lte-m-cat-tracker/kicad/lte-m-cat-tracker.kicad_sch (KiCad schematic)
At the start: 41 parts, among them J1 JST-PH-2mm-2P, J2 USB-C-16P, SW1 MSK12C02, U1 SIM7080G-M, U2 ESP32-C3FH4, U3 LIS2DW12TR, U4 TP4056, U5 XC6220B331MR-G, U6 TXB0104RGYR, Y1 40MHz_CL12pF_2016

Commit message: 回路図(修正⑦・U6/USB/CHIP_EN同期済み)をコミット固定＋KiCad起動時巻き戻り事故の記録と再発防止ルール
Co-Authored-By: Claude Fable 5 <noreply@anthropic.com>
Parts:
- added C20: 100nF, lte-m-custom:C_0402, symbol Device:C
- added R8: 10k, Resistor_SMD:R_0402_1005Metric, symbol Device:R
Connections:
- net +3.3V: now also R8.2
- net GND: now also C20.2
- net CHIP_EN: now reaches R5.1, U2.7 (CHIP_EN)
- net CHIP_EN: now also C20.1
- net USB_DP: now reaches J2.A6 (D+)
- net USB_DP: now also U2.26 (GPIO19)
- net USB_DN: now reaches J2.A7 (D-)
- net USB_DN: now also U2.25 (GPIO18)
- net ESP_GPIO2: now reaches U2.6 (GPIO2)
- net ESP_GPIO2: now also R8.1
- no-connect marks 31 -> 26
Changed lines of the file:
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@@
     (effects(font(size 1.27 1.27))(justify right))
 )
-  (no_connect (at 27.94 58.42))
-  (no_connect (at 27.94 55.88))
   (symbol (lib_id "power:GND") (at 27.94 45.72 0)(unit 1)
     (exclude_from_sim no)(in_bom no)(on_board no)
@@
     (effects(font(size 1.27 1.27))(justify right))
 )
-  (no_connect (at 66.04 180.34))
   (label "SIM_STATUS_33" (at 66.04 208.28 180)
     (effects(font(size 1.27 1.27))(justify right))
 )
-  (no_connect (at 66.04 193.04))
-  (no_connect (at 66.04 195.58))
   (no_connect (at 111.76 190.5))
   (no_connect (at 111.76 193.04))
@@
     (effects(font(size 1.27 1.27))(justify right))
 )
-)
+  (symbol (lib_id "Device:R") (at 62.23 180.34 270) (unit 1)
+    (exclude_from_sim no)(in_bom yes)(on_board yes)
+    (property "Reference" "R8" (at 62.23 176.84 0)(effects(font(size 1.27 1.27))))
+    (property "Value" "10k" (at 62.23 178.34 0)(effects(font(size 1.27 1.27))))
+    (property "Footprint" "Resistor_SMD:R_0402_1005Metric" (at 62.23 180.34 0)(effects(font(size 1.27 1.27))hide))
+    (property "LCSC" "C25744" (at 62.23 180.34 0)(effects(font(size 1.27 1.27))hide))
+  )
+  (symbol (lib_id "power:+3.3V") (at 58.42 180.34 0)(unit 1)
+    (exclude_from_sim no)(in_bom no)(on_board no)
+    (property "Reference" "#PWR"(at 58.42 177.8 0)(effects(font(size 1.27 1.27))hide))
+    (property "Value" "+3.3V"(at 58.42 179.07 0)(effects(font(size 1.27 1.27))))
+    (property "Footprint" ""(at 58.42 180.34 0)(effects(font(size 1.27 1.27))hide)))
+  (label "ESP_GPIO2" (at 66.04 180.34 180)
+    (effects(font(size 1.27 1.27))(justify right))
+)
+  (label "USB_DN" (at 66.04 193.04 180)
+    (effects(font(size 1.27 1.27))(justify right))
+)
+  (label "USB_DP" (at 66.04 195.58 180)
+    (effects(font(size 1.27 1.27))(justify right))
+)
+  (label "USB_DP" (at 27.94 55.88 180)
+    (effects(font(size 1.27 1.27))(justify right))
+)
+  (label "USB_DN" (at 27.94 58.42 180)
+    (effects(font(size 1.27 1.27))(justify right))
+)
+  (label "CHIP_EN" (at 111.76 185.42 0)
+    (effects(font(size 1.27 1.27))(justify left))
+)
+  (symbol (lib_id "Device:C") (at 127.0 189.23 0) (unit 1)
+    (exclude_from_sim no)(in_bom yes)(on_board yes)
+    (property "Reference" "C20" (at 129.54 187.95999999999998 0)(effects(font(size 1.27 1.27))))
+    (property "Value" "100nF" (at 129.54 190.5 0)(effects(font(size 1.27 1.27))))
+    (property "Footprint" "lte-m-custom:C_0402" (at 127.0 189.23 0)(effects(font(size 1.27 1.27))hide))
+    (property "LCSC" "C14663" (at 127.0 189.23 0)(effects(font(size 1.27 1.27))hide))
+  )
+  (label "CHIP_EN" (at 127.0 185.42 0)
+    (effects(font(size 1.27 1.27))(justify left))
+)
+  (symbol (lib_id "power:GND") (at 127.0 193.04 0)(unit 1)
+    (exclude_from_sim no)(in_bom no)(on_board no)
+    (property "Reference" "#PWR"(at 127.0 195.57999999999998 0)(effects(font(size 1.27 1.27))hide))
+    (property "Value" "GND"(at 127.0 194.31 0)(effects(font(size 1.27 1.27))))
+    (property "Footprint" ""(at 127.0 193.04 0)(effects(font(size 1.27 1.27))hide)))
+)
