File: lte-m-cat-tracker/kicad/lte-m-cat-tracker.kicad_sch (KiCad schematic)
At the start: 43 parts, among them J1 JST-PH-2mm-2P, J2 USB-C-16P, SW1 MSK12C02, U1 SIM7080G-M, U2 ESP32-C3FH4, U3 LIS2DW12TR, U4 TP4056, U5 XC6220B331MR-G, U6 TXB0104RGYR, Y1 40MHz_CL12pF_2016

Commit message: 回路図同期完了(修正㉒): B-2のピン変更9箇所を反映・netlist検証でPCBと完全一致・FW TODO7,8追記
Co-Authored-By: Claude Fable 5 <noreply@anthropic.com>
Connections:
- net SIM_STATUS_33 is gone; now on net SIM_RXD_33: U2.4 (XTAL_32K_P), U6.11 (B3)
- net SIM_RXD: now also U6.4 (A3); no longer U6.3 (A2)
- net SIM_RXD_33: no longer U2.28 (U0TXD), U6.12 (B2)
- net SIM_TXD_33: now also U2.12 (MTCK); no longer U2.27 (U0RXD)
- net SIM_STATUS: no longer names the net of U1.42 (STATUS)
- net SIM_STATUS: no longer U6.4 (A3)
- no-connect marks 26 -> 30
Changed lines of the file:
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@@
     (effects(font(size 1.27 1.27))(justify right))
 )
-  (label "SIM_STATUS" (at 218.44 88.9 180)
-    (effects(font(size 1.27 1.27))(justify right))
-)
+  (no_connect (at 218.44 88.9))
   (no_connect (at 218.44 91.44))
   (no_connect (at 218.44 93.98))
@@
     (effects(font(size 1.27 1.27))(justify left))
 )
-  (label "SIM_TXD_33" (at 66.04 203.2 180)
-    (effects(font(size 1.27 1.27))(justify right))
-)
-  (label "SIM_RXD_33" (at 66.04 200.66 180)
-    (effects(font(size 1.27 1.27))(justify right))
-)
+  (no_connect (at 66.04 203.2))
+  (no_connect (at 66.04 200.66))
   (label "I2C_SDA" (at 66.04 185.42 180)
     (effects(font(size 1.27 1.27))(justify right))
@@
     (effects(font(size 1.27 1.27))(justify right))
 )
-  (label "SIM_STATUS_33" (at 66.04 208.28 180)
+  (label "SIM_RXD_33" (at 66.04 208.28 180)
     (effects(font(size 1.27 1.27))(justify right))
 )
   (no_connect (at 111.76 190.5))
   (no_connect (at 111.76 193.04))
-  (no_connect (at 111.76 195.58))
+  (label "SIM_TXD_33" (at 111.76 195.58 0)
+    (effects(font(size 1.27 1.27))(justify left))
+)
   (no_connect (at 111.76 198.12))
   (no_connect (at 111.76 203.2))
@@
     (effects(font(size 1.27 1.27))(justify right))
 )
-  (label "SIM_RXD" (at 162.56 213.36 180)
-    (effects(font(size 1.27 1.27))(justify right))
-)
-  (label "SIM_STATUS" (at 162.56 215.9 180)
+  (no_connect (at 162.56 213.36))
+  (label "SIM_RXD" (at 162.56 215.9 180)
     (effects(font(size 1.27 1.27))(justify right))
 )
@@
     (effects(font(size 1.27 1.27))(justify left))
 )
-  (label "SIM_RXD_33" (at 193.04000000000002 213.36 0)
-    (effects(font(size 1.27 1.27))(justify left))
-)
-  (label "SIM_STATUS_33" (at 193.04000000000002 215.9 0)
-    (effects(font(size 1.27 1.27))(justify left))
-)
+  (no_connect (at 193.04000000000002 213.36))
+  (label "SIM_RXD_33" (at 193.04000000000002 215.9 0)
+    (effects(font(size 1.27 1.27))(justify left))
+)
